Commit message: UR5e Arm

File: ros2_ws/src/nora_description/urdf/materials.xacro (robot description, xacro)
@@ -1,8 +1,20 @@
 <?xml version="1.0" encoding="utf-8"?>
 <!--
-  materials.xacro — shared material definitions for the NORA arm.
+  materials.xacro — shared material definitions for the NORA / UR5e arm.
   Include this file at the top of any xacro that needs arm materials.
 -->
 <robot xmlns:xacro="http://www.ros.org/wiki/xacro">
+  <!-- Universal Robots classic blue -->
+  <material name="ur_blue">
+    <color rgba="0.18 0.38 0.60 1.0"/>
+  </material>
+  <!-- Universal Robots metallic grey body -->
+  <material name="ur_grey">
+    <color rgba="0.78 0.78 0.80 1.0"/>
+  </material>
+  <!-- Universal Robots joint collar dark grey -->
+  <material name="ur_dark">
+    <color rgba="0.22 0.22 0.25 1.0"/>
+  </material>
   <!-- Silver / metallic links -->
   <material name="silver">

File: ros2_ws/src/nora_description/urdf/nora_arm.urdf.xacro (robot description, xacro)
@@ -1,8 +1,19 @@
 <?xml version="1.0" encoding="utf-8"?>
 <!--
-  nora_arm.urdf.xacro
-  6-DOF NORA arm description using primitive geometries (no external meshes).
-  Macro layout:
-    world -> base_link -> link1 -> link2 -> link3 -> link4 -> link5 -> link6 -> gripper_link
+  nora_arm.urdf.xacro — Universal Robots UR5e 6-DOF Robotic Manipulator with Gripper.
+  Kinematic Chain:
+    world -> base_link
+          -> shoulder_link   (shoulder_pan_joint,  Z-axis yaw)
+          -> upper_arm_link   (shoulder_lift_joint, Y-axis pitch)
+          -> forearm_link     (elbow_joint,         Y-axis pitch)
+          -> wrist_1_link     (wrist_1_joint,       Y-axis pitch)
+          -> wrist_2_link     (wrist_2_joint,       Z-axis yaw)
+          -> wrist_3_link     (wrist_3_joint,       Y-axis pitch)
+          -> flange -> tool0 -> gripper_link (gripper_joint)
+  Specifications (UR5e Official):
+    Reach:              850 mm (0.85 m)
+    Payload:            5.0 kg
+    Total Arm Mass:     ~20.6 kg
+    Joint Velocities:   3.14 rad/s (joints 1-3), 6.28 rad/s (joints 4-6)
 -->
 <robot name="nora_arm" xmlns:xacro="http://www.ros.org/wiki/xacro">
@@ -13,21 +24,38 @@
   <xacro:include filename="$(find nora_description)/urdf/ros2_control.xacro"/>
   <!-- ===================================================================
-       Properties
-  ==================================================================== -->
-  <xacro:property name="joint_effort"   value="100.0"/>
-  <xacro:property name="joint_velocity" value="1.0"/>
-  <xacro:property name="joint_lower"    value="${-pi}"/>
-  <xacro:property name="joint_upper"    value="${pi}"/>
-  <!-- Simple diagonal inertia helper -->
-  <xacro:macro name="simple_inertia" params="mass ixx iyy izz">
+       UR5e Kinematic & Dynamic Parameters
+  ==================================================================== -->
+  <xacro:property name="d1" value="0.1625"/>   <!-- Base to shoulder Z -->
+  <xacro:property name="a2" value="0.4250"/>   <!-- Upper arm length -->
+  <xacro:property name="a3" value="0.3922"/>   <!-- Forearm length -->
+  <xacro:property name="d4" value="0.1333"/>   <!-- Wrist 1 offset Y -->
+  <xacro:property name="d5" value="0.0997"/>   <!-- Wrist 2 offset Z -->
+  <xacro:property name="d6" value="0.0996"/>   <!-- Wrist 3 offset Y -->
+  <!-- Joint limits -->
+  <xacro:property name="joint_lower"    value="${-2*pi}"/>
+  <xacro:property name="joint_upper"    value="${2*pi}"/>
+  <xacro:property name="joint_vel_arm"  value="3.14159"/>  <!-- 180 deg/s -->
+  <xacro:property name="joint_vel_wri"  value="6.28318"/>  <!-- 360 deg/s -->
+  <xacro:property name="joint_eff_arm"  value="150.0"/>
+  <xacro:property name="joint_eff_wri"  value="28.0"/>
+  <!-- Helper for box/cylinder inertia -->
+  <xacro:macro name="cylinder_inertia" params="m r h">
     <inertial>
-      <mass value="${mass}"/>
-      <inertia ixx="${ixx}" ixy="0.0" ixz="0.0"
-               iyy="${iyy}" iyz="0.0"
-               izz="${izz}"/>
+      <mass value="${m}"/>
+      <inertia ixx="${m*(3*r*r + h*h)/12}" ixy="0" ixz="0"
+               iyy="${m*(3*r*r + h*h)/12}" iyz="0"
+               izz="${m*r*r/2}"/>
     </inertial>
   </xacro:macro>
-  <!-- ===================================================================
-       World / Base
+  <xacro:macro name="box_inertia" params="m x y z">
+    <inertial>
+      <mass value="${m}"/>
+      <inertia ixx="${m*(y*y + z*z)/12}" ixy="0" ixz="0"
+               iyy="${m*(x*x + z*z)/12}" iyz="0"
+               izz="${m*(x*x + y*y)/12}"/>
+    </inertial>
+  </xacro:macro>
+  <!-- ===================================================================
+       World & Base Link
   ==================================================================== -->
   <link name="world"/>
@@ -37,181 +65,254 @@
     <origin xyz="0 0 0" rpy="0 0 0"/>
   </joint>
-  <!-- base_link: large cylinder as the mounting base -->
+  <!-- base_link: UR5e cylindrical base -->
   <link name="base_link">
-    <xacro:simple_inertia mass="2.0" ixx="0.02" iyy="0.02" izz="0.01"/>
-    <visual>
-      <origin xyz="0 0 0.05" rpy="0 0 0"/>
-      <geometry><cylinder radius="0.08" length="0.10"/></geometry>
-      <material name="dark_grey"/>
-    </visual>
-    <collision>
-      <origin xyz="0 0 0.05" rpy="0 0 0"/>
-      <geometry><cylinder radius="0.08" length="0.10"/></geometry>
-    </collision>
-  </link>
-  <!-- ===================================================================
-       Link 1 — shoulder yaw
-  ==================================================================== -->
-  <joint name="joint1" type="revolute">
+    <xacro:cylinder_inertia m="4.0" r="0.075" h="0.1625"/>
+    <visual>
+      <origin xyz="0 0 ${d1/2}" rpy="0 0 0"/>
+      <geometry><cylinder radius="0.075" length="${d1}"/></geometry>
+      <material name="ur_dark"/>
+    </visual>
+    <collision>
+      <origin xyz="0 0 ${d1/2}" rpy="0 0 0"/>
+      <geometry><cylinder radius="0.075" length="${d1}"/></geometry>
+    </collision>
+  </link>
+  <!-- ===================================================================
+       Joint 1: shoulder_pan_joint (Yaw)
+  ==================================================================== -->
+  <joint name="shoulder_pan_joint" type="revolute">
     <parent link="base_link"/>
+    <child  link="shoulder_link"/>
+    <origin xyz="0 0 ${d1}" rpy="0 0 0"/>
+    <axis xyz="0 0 1"/>
+    <limit lower="${joint_lower}" upper="${joint_upper}"
+           effort="${joint_eff_arm}" velocity="${joint_vel_arm}"/>
+    <dynamics damping="0.5" friction="0.1"/>
+  </joint>
+  <link name="shoulder_link">
+    <xacro:cylinder_inertia m="3.7" r="0.065" h="0.16"/>
+    <visual>
+      <origin xyz="0 0 0" rpy="0 0 0"/>
+      <geometry><cylinder radius="0.065" length="0.16"/></geometry>
+      <material name="ur_blue"/>
+    </visual>
+    <visual>
+      <origin xyz="0 0.05 0" rpy="${pi/2} 0 0"/>
+      <geometry><cylinder radius="0.06" length="0.12"/></geometry>
+      <material name="ur_grey"/>
+    </visual>
+    <collision>
+      <origin xyz="0 0 0" rpy="0 0 0"/>
+      <geometry><cylinder radius="0.065" length="0.16"/></geometry>
+    </collision>
+  </link>
+  <!-- ===================================================================
+       Joint 2: shoulder_lift_joint (Pitch)
+  ==================================================================== -->
+  <joint name="shoulder_lift_joint" type="revolute">
+    <parent link="shoulder_link"/>
+    <child  link="upper_arm_link"/>
+    <origin xyz="0 ${d4} 0" rpy="0 0 0"/>
+    <axis xyz="0 1 0"/>
+    <limit lower="${joint_lower}" upper="${joint_upper}"
+           effort="${joint_eff_arm}" velocity="${joint_vel_arm}"/>
+    <dynamics damping="0.5" friction="0.1"/>
+  </joint>
+  <link name="upper_arm_link">
+    <xacro:cylinder_inertia m="8.39" r="0.055" h="${a2}"/>
+    <!-- Upper arm main tube -->
+    <visual>
+      <origin xyz="0 0 ${a2/2}" rpy="0 0 0"/>
+      <geometry><cylinder radius="0.055" length="${a2}"/></geometry>
+      <material name="ur_grey"/>
+    </visual>
+    <!-- Upper arm joint cap -->
+    <visual>
+      <origin xyz="0 0 0" rpy="${pi/2} 0 0"/>
+      <geometry><cylinder radius="0.06" length="0.12"/></geometry>
+      <material name="ur_blue"/>
+    </visual>
+    <collision>
+      <origin xyz="0 0 ${a2/2}" rpy="0 0 0"/>
+      <geometry><cylinder radius="0.055" length="${a2}"/></geometry>
+    </collision>
+  </link>
+  <!-- ===================================================================
+       Joint 3: elbow_joint (Pitch)
+  ==================================================================== -->
+  <joint name="elbow_joint" type="revolute">
+    <parent link="upper_arm_link"/>
+    <child  link="forearm_link"/>
+    <origin xyz="0 -0.1197 ${a2}" rpy="0 0 0"/>
+    <axis xyz="0 1 0"/>
+    <limit lower="${joint_lower}" upper="${joint_upper}"
+           effort="${joint_eff_arm}" velocity="${joint_vel_arm}"/>
+    <dynamics damping="0.5" friction="0.1"/>
+  </joint>
+  <link name="forearm_link">
+    <xacro:cylinder_inertia m="2.275" r="0.045" h="${a3}"/>
+    <!-- Forearm tube -->
+    <visual>
+      <origin xyz="0 0 ${a3/2}" rpy="0 0 0"/>
+      <geometry><cylinder radius="0.045" length="${a3}"/></geometry>
+      <material name="ur_grey"/>
+    </visual>
+    <!-- Elbow joint cap -->
+    <visual>
+      <origin xyz="0 0 0" rpy="${pi/2} 0 0"/>
+      <geometry><cylinder radius="0.055" length="0.11"/></geometry>
+      <material name="ur_blue"/>
+    </visual>
+    <collision>
+      <origin xyz="0 0 ${a3/2}" rpy="0 0 0"/>
+      <geometry><cylinder radius="0.045" length="${a3}"/></geometry>
+    </collision>
+  </link>
+  <!-- ===================================================================
+       Joint 4: wrist_1_joint (Pitch)
+  ==================================================================== -->
+  <joint name="wrist_1_joint" type="revolute">
+    <parent link="forearm_link"/>
+    <child  link="wrist_1_link"/>
+    <origin xyz="0 0 ${a3}" rpy="0 0 0"/>
+    <axis xyz="0 1 0"/>
+    <limit lower="${joint_lower}" upper="${joint_upper}"
+           effort="${joint_eff_wri}" velocity="${joint_vel_wri}"/>
+    <dynamics damping="0.2" friction="0.05"/>
+  </joint>
+  <link name="wrist_1_link">
+    <xacro:cylinder_inertia m="1.219" r="0.04" h="${d5}"/>
+    <visual>
+      <origin xyz="0 ${d5/2} 0" rpy="${pi/2} 0 0"/>
+      <geometry><cylinder radius="0.04" length="${d5}"/></geometry>
+      <material name="ur_blue"/>
+    </visual>
+    <collision>
+      <origin xyz="0 ${d5/2} 0" rpy="${pi/2} 0 0"/>
+      <geometry><cylinder radius="0.04" length="${d5}"/></geometry>
+    </collision>
+  </link>
+  <!-- ===================================================================
+       Joint 5: wrist_2_joint (Yaw)
+  ==================================================================== -->
+  <joint name="wrist_2_joint" type="revolute">
+    <parent link="wrist_1_link"/>
+    <child  link="wrist_2_link"/>
+    <origin xyz="0 ${d5} 0" rpy="0 0 0"/>
+    <axis xyz="0 0 1"/>
+    <limit lower="${joint_lower}" upper="${joint_upper}"
+           effort="${joint_eff_wri}" velocity="${joint_vel_wri}"/>
+    <dynamics damping="0.2" friction="0.05"/>
+  </joint>
+  <link name="wrist_2_link">
+    <xacro:cylinder_inertia m="1.219" r="0.038" h="${d5}"/>
+    <visual>
+      <origin xyz="0 0 ${d5/2}" rpy="0 0 0"/>
+      <geometry><cylinder radius="0.038" length="${d5}"/></geometry>
+      <material name="ur_grey"/>
+    </visual>
+    <collision>
+      <origin xyz="0 0 ${d5/2}" rpy="0 0 0"/>
+      <geometry><cylinder radius="0.038" length="${d5}"/></geometry>
+    </collision>
+  </link>
+  <!-- ===================================================================
+       Joint 6: wrist_3_joint (Pitch)
+  ==================================================================== -->
+  <joint name="wrist_3_joint" type="revolute">
+    <parent link="wrist_2_link"/>
+    <child  link="wrist_3_link"/>
+    <origin xyz="0 0 ${d5}" rpy="0 0 0"/>
+    <axis xyz="0 1 0"/>
+    <limit lower="${joint_lower}" upper="${joint_upper}"
+           effort="${joint_eff_wri}" velocity="${joint_vel_wri}"/>
+    <dynamics damping="0.2" friction="0.05"/>
+  </joint>
+  <link name="wrist_3_link">
+    <xacro:cylinder_inertia m="0.188" r="0.035" h="${d6}"/>
+    <visual>
+      <origin xyz="0 ${d6/2} 0" rpy="${pi/2} 0 0"/>
+      <geometry><cylinder radius="0.035" length="${d6}"/></geometry>
+      <material name="ur_blue"/>
+    </visual>
+    <collision>
+      <origin xyz="0 ${d6/2} 0" rpy="${pi/2} 0 0"/>
+      <geometry><cylinder radius="0.035" length="${d6}"/></geometry>
+    </collision>
+  </link>
+  <!-- ===================================================================
+       Tool Flange & tool0 Frame
+  ==================================================================== -->
+  <joint name="wrist_3_to_flange" type="fixed">
+    <parent link="wrist_3_link"/>
+    <child  link="flange"/>
+    <origin xyz="0 ${d6} 0" rpy="0 0 0"/>
+  </joint>
+  <link name="flange">
+    <visual>
+      <origin xyz="0 0.005 0" rpy="${pi/2} 0 0"/>
+      <geometry><cylinder radius="0.035" length="0.01"/></geometry>
+      <material name="ur_dark"/>
+    </visual>
+  </link>
+  <joint name="flange_to_tool0" type="fixed">
+    <parent link="flange"/>
+    <child  link="tool0"/>
+    <origin xyz="0 0.01 0" rpy="${-pi/2} 0 0"/>
+  </joint>
+  <link name="tool0"/>
+  <!-- ===================================================================
+       End-Effector / Parallel Gripper
+  ==================================================================== -->
+  <joint name="gripper_joint" type="prismatic">
+    <parent link="tool0"/>
+    <child  link="gripper_link"/>
+    <origin xyz="0 0 0.05" rpy="0 0 0"/>
+    <axis xyz="0 1 0"/>
+    <limit lower="0.0" upper="0.08" effort="50.0" velocity="0.5"/>
+    <dynamics damping="0.1" friction="0.02"/>
+  </joint>
+  <link name="gripper_link">
+    <xacro:box_inertia m="0.3" x="0.06" y="0.10" z="0.08"/>
+    <!-- Gripper Palm -->
+    <visual>
+      <origin xyz="0 0 0.02" rpy="0 0 0"/>
+      <geometry><box size="0.05 0.08 0.04"/></geometry>
+      <material name="ur_dark"/>
+    </visual>
+    <!-- Gripper Fingers -->
+    <visual>
+      <origin xyz="0 0.035 0.055" rpy="0 0 0"/>
+      <geometry><box size="0.025 0.015 0.05"/></geometry>
+      <material name="orange"/>
+    </visual>
+    <visual>
+      <origin xyz="0 -0.035 0.055" rpy="0 0 0"/>
+      <geometry><box size="0.025 0.015 0.05"/></geometry>
+      <material name="orange"/>
+    </visual>
+    <collision>
+      <origin xyz="0 0 0.035" rpy="0 0 0"/>
+      <geometry><box size="0.05 0.09 0.07"/></geometry>
+    </collision>
+  </link>
+  <!-- ===================================================================
+       Backwards Compatibility Aliases (link1..link6)
+  ==================================================================== -->
+  <joint name="alias_link1" type="fixed">
+    <parent link="shoulder_link"/>
     <child  link="link1"/>
-    <origin xyz="0 0 0.10" rpy="0 0 0"/>
-    <axis xyz="0 0 1"/>
-    <limit lower="${joint_lower}" upper="${joint_upper}"
-           effort="${joint_effort}" velocity="${joint_velocity}"/>
-  </joint>
-  <link name="link1">
-    <xacro:simple_inertia mass="1.0" ixx="0.01" iyy="0.01" izz="0.005"/>
-    <visual>
-      <origin xyz="0 0 0.075" rpy="0 0 0"/>
-      <geometry><box size="0.07 0.07 0.15"/></geometry>
-      <material name="silver"/>
-    </visual>
-    <collision>
-      <origin xyz="0 0 0.075" rpy="0 0 0"/>
-      <geometry><box size="0.07 0.07 0.15"/></geometry>
-    </collision>
-  </link>
-  <!-- ===================================================================
-       Link 2 — shoulder pitch
-  ==================================================================== -->
-  <joint name="joint2" type="revolute">
-    <parent link="link1"/>
-    <child  link="link2"/>
-    <origin xyz="0 0 0.15" rpy="0 0 0"/>
-    <axis xyz="0 1 0"/>
-    <limit lower="${joint_lower}" upper="${joint_upper}"
-           effort="${joint_effort}" velocity="${joint_velocity}"/>
-  </joint>
-  <link name="link2">
-    <xacro:simple_inertia mass="1.0" ixx="0.01" iyy="0.005" izz="0.01"/>
-    <visual>
-      <origin xyz="0 0 0.10" rpy="0 0 0"/>
-      <geometry><cylinder radius="0.04" length="0.20"/></geometry>
-      <material name="silver"/>
-    </visual>
-    <collision>
-      <origin xyz="0 0 0.10" rpy="0 0 0"/>
-      <geometry><cylinder radius="0.04" length="0.20"/></geometry>
-    </collision>
-  </link>
-  <!-- ===================================================================
-       Link 3 — elbow pitch
-  ==================================================================== -->
-  <joint name="joint3" type="revolute">
-    <parent link="link2"/>
-    <child  link="link3"/>
-    <origin xyz="0 0 0.20" rpy="0 0 0"/>
-    <axis xyz="0 1 0"/>
-    <limit lower="${joint_lower}" upper="${joint_upper}"
-           effort="${joint_effort}" velocity="${joint_velocity}"/>
-  </joint>
-  <link name="link3">
-    <xacro:simple_inertia mass="1.0" ixx="0.008" iyy="0.004" izz="0.008"/>
-    <visual>
-      <origin xyz="0 0 0.09" rpy="0 0 0"/>
-      <geometry><cylinder radius="0.035" length="0.18"/></geometry>
-      <material name="silver"/>
-    </visual>
-    <collision>
-      <origin xyz="0 0 0.09" rpy="0 0 0"/>
-      <geometry><cylinder radius="0.035" length="0.18"/></geometry>
-    </collision>
-  </link>
-  <!-- ===================================================================
-       Link 4 — forearm roll
-  ==================================================================== -->
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
File: ros2_ws/src/nora_description/urdf/ros2_control.xacro (robot description, xacro)
@@ -1,9 +1,5 @@
 <?xml version="1.0" encoding="utf-8"?>
 <!--
-  ros2_control.xacro — ros2_control hardware interface stub for the NORA arm.
-  Defines a <ros2_control> block for a joint_trajectory_controller with
-  PositionJointInterface for all 6 arm joints and the gripper joint.
-  # TODO(nora): Replace mock hardware plugin with real driver once available.
-  # TODO(nora): Add velocity/effort command interfaces as needed.
+  ros2_control.xacro — ros2_control hardware interface for UR5e manipulator.
 -->
 <robot xmlns:xacro="http://www.ros.org/wiki/xacro">
@@ -11,58 +7,56 @@
     <ros2_control name="${name}" type="system">
       <!-- ----------------------------------------------------------------
-           Hardware plugin (mock for simulation; swap for real driver)
+           Hardware plugin (mock for simulation/dev; swap for ur_robot_driver)
       ---------------------------------------------------------------- -->
       <hardware>
-        <!-- TODO(nora): replace with actual driver plugin, e.g.
-             <plugin>nora_hardware/NoraArmHardware</plugin> -->
         <plugin>mock_components/GenericSystem</plugin>
       </hardware>
       <!-- ----------------------------------------------------------------
-           Arm joints — position command + state interfaces
+           UR5e 6-DOF Arm Joints
       ---------------------------------------------------------------- -->
-      <joint name="joint1">
+      <joint name="shoulder_pan_joint">
         <command_interface name="position">
-          <param name="min">${-pi}</param>
-          <param name="max">${pi}</param>
+          <param name="min">${-2*pi}</param>
+          <param name="max">${2*pi}</param>
         </command_interface>
         <state_interface name="position"/>
         <state_interface name="velocity"/>
       </joint>
-      <joint name="joint2">
+      <joint name="shoulder_lift_joint">
         <command_interface name="position">
-          <param name="min">${-pi}</param>
-          <param name="max">${pi}</param>
+          <param name="min">${-2*pi}</param>
+          <param name="max">${2*pi}</param>
         </command_interface>
         <state_interface name="position"/>
         <state_interface name="velocity"/>
       </joint>
-      <joint name="joint3">
+      <joint name="elbow_joint">
         <command_interface name="position">
-          <param name="min">${-pi}</param>
-          <param name="max">${pi}</param>
+          <param name="min">${-2*pi}</param>
+          <param name="max">${2*pi}</param>
         </command_interface>
         <state_interface name="position"/>
         <state_interface name="velocity"/>
       </joint>
-      <joint name="joint4">
+      <joint name="wrist_1_joint">
         <command_interface name="position">
-          <param name="min">${-pi}</param>
-          <param name="max">${pi}</param>
+          <param name="min">${-2*pi}</param>
+          <param name="max">${2*pi}</param>
         </command_interface>
         <state_interface name="position"/>
         <state_interface name="velocity"/>
       </joint>
-      <joint name="joint5">
+      <joint name="wrist_2_joint">
         <command_interface name="position">
-          <param name="min">${-pi}</param>
-          <param name="max">${pi}</param>
+          <param name="min">${-2*pi}</param>
+          <param name="max">${2*pi}</param>
         </command_interface>
         <state_interface name="position"/>
         <state_interface name="velocity"/>
       </joint>
-      <joint name="joint6">
+      <joint name="wrist_3_joint">
         <command_interface name="position">
-          <param name="min">${-pi}</param>
-          <param name="max">${pi}</param>
+          <param name="min">${-2*pi}</param>
+          <param name="max">${2*pi}</param>
         </command_interface>
         <state_interface name="position"/>
@@ -70,5 +64,5 @@
       </joint>
       <!-- ----------------------------------------------------------------
-           Gripper joint
+           Gripper Joint
       ---------------------------------------------------------------- -->
       <joint name="gripper_joint">
