Commit message: Add RealSense D435 camera frames, 3D optical projection, and multi-object tracking for perception

File: frontend/public/nora_arm.urdf (robot description, URDF)
Before this commit: robot nora_arm, 10 links, 9 joints
Links:
- added link camera_color_frame
- added link camera_color_optical_frame
- added link camera_depth_frame
- added link camera_depth_optical_frame
- added link camera_link; collision box size=0.09 0.025 0.025; visual box size=0.09 0.025 0.025
Joints:
- added joint camera_color_joint: type fixed, parent camera_link, child camera_color_frame, origin xyz=0.015 0 0 rpy=0 0 0
- added joint camera_color_optical_joint: type fixed, parent camera_color_frame, child camera_color_optical_frame, origin xyz=0 0 0 rpy=-1.5707963 0 -1.5707963
- added joint camera_depth_joint: type fixed, parent camera_link, child camera_depth_frame, origin xyz=-0.015 0 0 rpy=0 0 0
- added joint camera_depth_optical_joint: type fixed, parent camera_depth_frame, child camera_depth_optical_frame, origin xyz=0 0 0 rpy=-1.5707963 0 -1.5707963
- added joint camera_mount_joint: type fixed, parent gripper_link, child camera_link, origin xyz=0 0.038 0.02 rpy=0 0 0

File: ros2_ws/src/nora_description/urdf/nora_arm.urdf.xacro (robot description, xacro)
@@ -298,4 +298,48 @@
   </link>
   <!-- ===================================================================
+       Eye-in-Hand RGB-D Camera (Intel RealSense D435) for Foxglove & ROS 2
+  ==================================================================== -->
+  <joint name="camera_mount_joint" type="fixed">
+    <parent link="gripper_link"/>
+    <child  link="camera_link"/>
+    <origin xyz="0 0.038 0.02" rpy="0 0 0"/>
+  </joint>
+  <link name="camera_link">
+    <xacro:box_inertia m="0.072" x="0.09" y="0.025" z="0.025"/>
+    <visual>
+      <origin xyz="0 0 0" rpy="0 0 0"/>
+      <geometry><box size="0.09 0.025 0.025"/></geometry>
+      <material name="ur_dark"/>
+    </visual>
+    <collision>
+      <origin xyz="0 0 0" rpy="0 0 0"/>
+      <geometry><box size="0.09 0.025 0.025"/></geometry>
+    </collision>
+  </link>
+  <joint name="camera_color_joint" type="fixed">
+    <parent link="camera_link"/>
+    <child  link="camera_color_frame"/>
+    <origin xyz="0.015 0 0" rpy="0 0 0"/>
+  </joint>
+  <link name="camera_color_frame"/>
+  <joint name="camera_color_optical_joint" type="fixed">
+    <parent link="camera_color_frame"/>
+    <child  link="camera_color_optical_frame"/>
+    <origin xyz="0 0 0" rpy="${-pi/2} 0 ${-pi/2}"/>
+  </joint>
+  <link name="camera_color_optical_frame"/>
+  <joint name="camera_depth_joint" type="fixed">
+    <parent link="camera_link"/>
+    <child  link="camera_depth_frame"/>
+    <origin xyz="-0.015 0 0" rpy="0 0 0"/>
+  </joint>
+  <link name="camera_depth_frame"/>
+  <joint name="camera_depth_optical_joint" type="fixed">
+    <parent link="camera_depth_frame"/>
+    <child  link="camera_depth_optical_frame"/>
+    <origin xyz="0 0 0" rpy="${-pi/2} 0 ${-pi/2}"/>
+  </joint>
+  <link name="camera_depth_optical_frame"/>
+  <!-- ===================================================================
        Backwards Compatibility Aliases (link1..link6)
   ==================================================================== -->
